File: USB-TouCAN.kicad_pcb (KiCad board)
At the start: 4 copper layers, 76.5 x 30.9 mm, 58 parts, among them J1 Conn_01x17_Pin, J10 CAN, J2 NC, J3 Conn_01x17_Pin, J4 USB2.0_16P, J5 Boot, J6 NC, J7 DE9_Receptacle, J8 RS-485/422-TX, J9 RS-422-RX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

Commit message: Cleanup after PCB review
Parts:
- C4, C7: value 18pF -> 15pF
- moved R19 1.32 mm to (169.7, 79.0)
- moved C13 0.18 mm to (158.7, 79.1)
- moved D1 0.10 mm to (160.9, 78.9)
- moved C9 0.09 mm to (183.0, 79.5)
Routing:
- net Net-(D2-A): track 1.35 -> 2.67 mm
- net /PB7: track 66.3 -> 65.0 mm
- net /CAN_L: track 15.4 -> 14.5 mm
- net /PC13: track 74.9 -> 74.3 mm
- net /PB13: track 21.4 -> 20.7 mm
- net /422_RE: track 66.7 -> 66.1 mm
- net /CAN_H: track 16.5 -> 16.0 mm
- net GND: track 36.4 -> 36.7 mm, vias 64 -> 67
