File: USB-TouCAN.kicad_sch (KiCad schematic)
At the start: 58 parts, among them J1 Conn_01x17_Pin, J10 CAN, J2 NC, J3 Conn_01x17_Pin, J4 USB2.0_16P, J5 Boot, J6 NC, J7 DE9_Receptacle, J8 RS-485/422-TX, J9 RS-422-RX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

Commit message: Cleanup after PCB review
Parts:
- C4, C7: value 18pF -> 15pF; LCSC C1549 -> C1548
Changed lines of the file:
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@@
 	)
 	(junction
+		(at 59.69 60.96)
+		(diameter 0)
+		(color 0 0 0 0)
+	)
+	(junction
 		(at 273.05 158.75)
 		(diameter 0)
@@
 	(wire
 		(pts
+			(xy 59.69 60.96) (xy 62.23 60.96)
+		)
+		(stroke
+			(width 0)
+			(type default)
+		)
+	)
+	(wire
+		(pts
 			(xy 180.34 49.53) (xy 180.34 55.88)
 		)
@@
 	(wire
 		(pts
+			(xy 59.69 55.88) (xy 59.69 60.96)
+		)
+		(stroke
+			(width 0)
+			(type default)
+		)
+	)
+	(wire
+		(pts
 			(xy 33.02 25.4) (xy 33.02 30.48)
 		)
@@
 	(wire
 		(pts
-			(xy 58.42 60.96) (xy 62.23 60.96)
+			(xy 58.42 60.96) (xy 59.69 60.96)
 		)
 		(stroke
@@
 	)
 	(symbol
+		(lib_id "power:PWR_FLAG")
+		(at 59.69 55.88 0)
+		(unit 1)
+		(exclude_from_sim no)
+		(in_bom yes)
+		(on_board yes)
+		(dnp no)
+		(fields_autoplaced yes)
+		(property "Reference" "#FLG01"
+			(at 59.69 53.975 0)
+			(effects
+				(font
+					(size 1.27 1.27)
+				)
+				(hide yes)
+			)
+		)
+		(property "Value" "PWR_FLAG"
+			(at 59.69 50.8 0)
+			(effects
+				(font
+					(size 1.27 1.27)
+				)
+			)
+		)
+		(property "Footprint" ""
+			(at 59.69 55.88 0)
+			(effects
+				(font
+					(size 1.27 1.27)
+				)
+				(hide yes)
+			)
+		)
+		(property "Datasheet" "~"
+			(at 59.69 55.88 0)
+			(effects
+				(font
+					(size 1.27 1.27)
+				)
+				(hide yes)
+			)
+		)
+		(property "Description" "Special symbol for telling ERC where power comes from"
+			(at 59.69 55.88 0)
+			(effects
+				(font
+					(size 1.27 1.27)
+				)
+				(hide yes)
+			)
+		)
+		(pin "1"
+		)
+		(instances
+			(project ""
+				(path "/26096f25-a87e-4f6d-a99b-624957e9ad57"
+					(reference "#FLG01")
+					(unit 1)
+				)
+			)
+		)
+	)
+	(symbol
 		(lib_id "power:GND")
 		(at 212.09 158.75 0)
@@
 			)
 		)
-		(property "Value" "18pF"
+		(property "Value" "15pF"
 			(at 176.53 67.818 90)
 			(effects
@@
 			)
 		)
-		(property "LCSC" "C1549"
+		(property "LCSC" "C1548"
 			(at 171.45 69.85 0)
 			(effects
@@
 			)
 		)
-		(property "Value" "18pF"
+		(property "Value" "15pF"
 			(at 176.53 62.738 90)
 			(effects
@@
 			)
 		)
-		(property "LCSC" "C1549"
+		(property "LCSC" "C1548"
 			(at 171.45 64.77 0)
 			(effects
