File: USB-FalCAN.kicad_pcb (KiCad board)
At the start: 4 copper layers, 76.5 x 30.9 mm, 59 parts, among them J1 Conn_01x17_Pin, J10 CAN, J2 NC, J3 Conn_01x17_Pin, J4 USB2.0_16P, J5 Boot, J6 NC, J7 DE9_Receptacle, J8 RS-485/422-TX, J9 RS-422-RX, SW3 BTN, U1 STM32F042C6Tx, U2 SN65HVD230, U3 SP3485EN, U4 SP3485EN, U5 MIC5504-3.3YM5, Y1 8MHz, Y2 32768Hz

Commit message: feat: Change to male D-sub, fix "B3" silk
Parts:
- J7: footprint Connector_Dsub:DSUB-9_Female_Horizontal_P2.77x2.84mm_EdgePinOffset7.70mm_Housed_MountingHolesOffset9.12mm -> Connector_Dsub:DSUB-9_Pins_Horizontal_P2.77x2.84mm_EdgePinOffset7.70mm_Housed_MountingHolesOffset9.12mm
- moved J7 11.1 mm to (142.1, 67.7)
Routing:
- net Net-(J7-PAD): track 35.2 -> 39.6 mm
- net /CAN_L: track 14.5 -> 17.0 mm
- net /CAN_H: track 16.0 -> 18.0 mm
Other:
- board text added: "B3"
